File: Full_Board/MSP_Subsystem/MSP432E401Y.kicad_sch (KiCad schematic)
At the start: 4 parts, among them J1-J3 Conn_01x10, J4-J2 Conn_01x10, J5-J7 Conn_01x10, J8-J6 Conn_01x10

Commit message: Fixed entire BOM for all components
Parts:
- J1-J3, J4-J2, J5-J7, J8-J6: Digikey Part Number (none) -> S7078-ND; Digikey link (none) -> https://www.digikey.com/en/products/detail/sullins-connecto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; Manufacturer's Part Number (none) -> PPTC102LFBN-RC; Mouser Part Number (none) -> 855-M50-3001045; Mouser link (none) -> https://www.mouser.com/ProductDetail/Harwin/M50-3001045?qs=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
Changed lines of the file:
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@@
+      (effects (font (size 1.27 1.27)) hide)
+    )
+    (property "Digikey Part Number" "S7078-ND" (id 4) (at 167.64 71.12 0)
+      (effects (font (size 1.27 1.27)) hide)
+    )
+    (property "Digikey link" "https://www.digikey.com/en/products/detail/sullins-connector-solutions/PPTC102LFBN-RC/810216" (id 5) (at 167.64 71.12 0)
+      (effects (font (size 1.27 1.27)) hide)
+    )
+    (property "Manufacturer's Part Number" "PPTC102LFBN-RC" (id 6) (at 167.64 71.12 0)
+      (effects (font (size 1.27 1.27)) hide)
+    )
+    (property "Mouser Part Number" "855-M50-3001045" (id 7) (at 167.64 71.12 0)
+      (effects (font (size 1.27 1.27)) hide)
+    )
+    (property "Mouser link" "https://www.mouser.com/ProductDetail/Harwin/M50-3001045?qs=sGAEpiMZZMvlX3nhDDO4ACiIlPQK9Fd3x0shJJA6fS8%3D" (id 8) (at 167.64 71.12 0)
       (effects (font (size 1.27 1.27)) hide)
     )
@@
       (effects (font (size 1.27 1.27)) hide)
     )
+    (property "Digikey Part Number" "S7078-ND" (id 4) (at 113.03 116.84 0)
+      (effects (font (size 1.27 1.27)) hide)
+    )
+    (property "Digikey link" "https://www.digikey.com/en/products/detail/sullins-connector-solutions/PPTC102LFBN-RC/810216" (id 5) (at 113.03 116.84 0)
+      (effects (font (size 1.27 1.27)) hide)
+    )
+    (property "Manufacturer's Part Number" "PPTC102LFBN-RC" (id 6) (at 113.03 116.84 0)
+      (effects (font (size 1.27 1.27)) hide)
+    )
+    (property "Mouser Part Number" "855-M50-3001045" (id 7) (at 113.03 116.84 0)
+      (effects (font (size 1.27 1.27)) hide)
+    )
+    (property "Mouser link" "https://www.mouser.com/ProductDetail/Harwin/M50-3001045?qs=sGAEpiMZZMvlX3nhDDO4ACiIlPQK9Fd3x0shJJA6fS8%3D" (id 8) (at 113.03 116.84 0)
+      (effects (font (size 1.27 1.27)) hide)
+    )
     (pin "1")
     (pin "10")
@@
     )
     (property "Datasheet" "~" (id 3) (at 168.91 116.84 0)
+      (effects (font (size 1.27 1.27)) hide)
+    )
+    (property "Digikey Part Number" "S7078-ND" (id 4) (at 168.91 116.84 0)
+      (effects (font (size 1.27 1.27)) hide)
+    )
+    (property "Digikey link" "https://www.digikey.com/en/products/detail/sullins-connector-solutions/PPTC102LFBN-RC/810216" (id 5) (at 168.91 116.84 0)
+      (effects (font (size 1.27 1.27)) hide)
+    )
+    (property "Manufacturer's Part Number" "PPTC102LFBN-RC" (id 6) (at 168.91 116.84 0)
+      (effects (font (size 1.27 1.27)) hide)
+    )
+    (property "Mouser Part Number" "855-M50-3001045" (id 7) (at 168.91 116.84 0)
+      (effects (font (size 1.27 1.27)) hide)
+    )
+    (property "Mouser link" "https://www.mouser.com/ProductDetail/Harwin/M50-3001045?qs=sGAEpiMZZMvlX3nhDDO4ACiIlPQK9Fd3x0shJJA6fS8%3D" (id 8) (at 168.91 116.84 0)
       (effects (font (size 1.27 1.27)) hide)
     )
@@
       (effects (font (size 1.27 1.27)) hide)
     )
+    (property "Digikey Part Number" "S7078-ND" (id 4) (at 111.76 71.12 0)
+      (effects (font (size 1.27 1.27)) hide)
+    )
+    (property "Digikey link" "https://www.digikey.com/en/products/detail/sullins-connector-solutions/PPTC102LFBN-RC/810216" (id 5) (at 111.76 71.12 0)
+      (effects (font (size 1.27 1.27)) hide)
+    )
+    (property "Manufacturer's Part Number" "PPTC102LFBN-RC" (id 6) (at 111.76 71.12 0)
+      (effects (font (size 1.27 1.27)) hide)
+    )
+    (property "Mouser Part Number" "855-M50-3001045" (id 7) (at 111.76 71.12 0)
+      (effects (font (size 1.27 1.27)) hide)
+    )
+    (property "Mouser link" "https://www.mouser.com/ProductDetail/Harwin/M50-3001045?qs=sGAEpiMZZMvlX3nhDDO4ACiIlPQK9Fd3x0shJJA6fS8%3D" (id 8) (at 111.76 71.12 0)
+      (effects (font (size 1.27 1.27)) hide)
+    )
