File: BareBones_Chess_Board/8x1/8x1.kicad_pcb (KiCad board)
At the start: 2 copper layers, 46.8 x 406.4 mm, 0 parts

Commit message: Fixed ground
Routing:
- net Top: track 387.1 -> 777.9 mm
- net GND: track 359.5 -> 0.00 mm, vias 8 -> 0
- net GND_8: track 0.00 -> 0.01 mm, vias 0 -> 1
- net GND_7: vias 0 -> 1
- net GND_6: vias 0 -> 1
- net GND_5: vias 0 -> 1
- net GND_4: vias 0 -> 1
- net GND_3: vias 0 -> 1
- net GND_2: vias 0 -> 1
- net GND_1: vias 0 -> 1
- added copper zone on B.Cu, net GND_1
- added copper zone on B.Cu, net GND_2
- added copper zone on B.Cu, net GND_3
- added copper zone on B.Cu, net GND_4
- added copper zone on B.Cu, net GND_5
- added copper zone on B.Cu, net GND_6
- added copper zone on B.Cu, net GND_7
- added copper zone on B.Cu, net GND_8
- added copper zone on F.Cu, net Top
