File: Boards/Main_Board/Electromagnet_Subsystem/Electromagnet.kicad_sch (KiCad schematic)
At the start: 5 parts, among them IC5 BD62130AEFJ-E2

Commit message: Correct spacing on sensor board, refactor datasheets and project libraries
Parts:
- C35: symbol CL10B104KB8NNC:CL10B104KB8NNNC -> CL10B104KB8NNNC:CL10B104KB8NNNC
Changed lines of the file:
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@@
     (pin "")
   )
-  (symbol (lib_id "CL10B104KB8NNC:CL10B104KB8NNNC") (at 133.35 99.06 90) (mirror x) (unit 1)
+  (symbol (lib_id "CL10B104KB8NNNC:CL10B104KB8NNNC") (at 133.35 99.06 90) (mirror x) (unit 1)
     (in_bom yes) (on_board yes)
     (property "Reference" "C35" (id 0) (at 139.7 101.6 90)
