File: Boards/Sensor_Board_2x16/_Top_Level/Sensor_Board_2x16.kicad_pcb (KiCad board)
At the start: 2 copper layers, 50.8 x 406.4 mm, 25 parts, among them J1 OQ0212500000G, J10 OQ0212500000G, J11 OQ0212500000G, J12 OQ0212500000G, J13 OQ0212500000G, J14 OQ0212500000G, J15 OQ0212500000G, J16 OQ0212500000G, J17 OQ0212500000G, J2 OQ0212500000G, J3 OQ0212500000G, J4 OQ0212500000G, J5 OQ0212500000G, J6 OQ0212500000G, J7 OQ0212500000G, J8 OQ0212500000G, J9 OQ0212500000G

Commit message: Correct spacing on sensor board, refactor datasheets and project libraries
Parts:
- moved S7 12.9 mm to (32.6, 360.8)
- moved S6 12.8 mm to (32.6, 313.2)
- moved S8 12.8 mm to (32.6, 408.4)
- moved S5 12.7 mm to (32.6, 265.6)
- moved S4 12.6 mm to (32.6, 217.9)
- moved S2 12.4 mm to (32.6, 122.7)
- moved S3 12.2 mm to (32.6, 170.3)
- moved S1 10.9 mm to (32.6, 75.0)
- moved J13 6.80 mm to (65.7, 201.3)
- moved J15 6.80 mm to (65.7, 296.0)
- moved J17 6.80 mm to (65.7, 390.7)
- moved J11 6.80 mm to (65.7, 106.6)
- moved J10 6.80 mm to (65.7, 59.3)
- moved J12 6.80 mm to (65.7, 154.0)
- moved J14 6.80 mm to (65.7, 248.7)
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Routing:
- net Net-(S1-Pad1): track 778.4 -> 758.8 mm
- net Net-(J15-Pad2): track 50.7 -> 56.6 mm
- net Net-(J16-Pad2): track 51.0 -> 56.9 mm
- net Net-(J17-Pad2): track 51.5 -> 57.2 mm
- net Net-(J14-Pad2): track 50.5 -> 56.1 mm
- net Net-(J13-Pad2): track 50.2 -> 55.7 mm
- net Net-(J11-Pad2): track 49.8 -> 55.0 mm
- net Net-(J12-Pad2): track 50.3 -> 55.4 mm
- net Net-(J10-Pad1): track 40.8 -> 37.2 mm
- net Net-(J16-Pad1): track 40.6 -> 37.2 mm
- net Net-(J17-Pad1): track 40.6 -> 37.2 mm
- net Net-(J15-Pad1): track 40.6 -> 37.2 mm
- net Net-(J13-Pad1): track 40.6 -> 37.2 mm
- net Net-(J11-Pad1): track 40.6 -> 37.2 mm
- net Net-(J14-Pad1): track 40.6 -> 37.2 mm
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Other:
- board size 50.8 x 406.4 mm -> 47.6 x 406.4 mm
