File: Boards/Main_Board/_Top_Level/Main_Board.kicad_pcb (KiCad board)
At the start: 2 copper layers, 174 x 97.8 mm, 229 parts, among them IC1 DRV8824QPWPRQ1, IC2 DRV8824QPWPRQ1, IC3 DRV8824QPWPRQ1, IC4 LM2576HVS-5.0_NOPB, IC5 BD62130AEFJ-E2, J1 302-S101, J1-J1 Conn_01x10, J10 KLDHCX-8-0202-A, J11 OQ0212500000G, J12 OQ0432500000G, J13 OQ0432500000G, J14 OQ0432500000G, J15 OQ0432500000G, J16 OQ0432500000G, J17 OQ0432500000G, J18 OQ0432500000G, J19 OQ0432500000G, J2 OQ0212500000G, J20 OQ0212500000G, J21 OQ0212500000G, J22 OQ0212500000G, J23 OQ0212500000G, J24 OQ0212500000G, J3 OQ0432500000G, J4 OQ0432500000G, J4-J1 Conn_01x10, J5 OQ0432500000G, J5-J1 Conn_01x10, J7 OQ0212500000G, J8 OQ0212500000G, J8-J1 Conn_01x10, J9 OQ0212500000G, U1 UCLAMP3301H.TCT, U10 LM2576SX-3.3-NOPB, U11 UCLAMP3301H.TCT, U12 UCLAMP3301H.TCT, U13 UCLAMP3301H.TCT, U14 UCLAMP3301H.TCT, U15 SN74LV4051ATPWRQ1, U16 SN74LV4051ATPWRQ1, U17 UCLAMP3301H.TCT, U18 UCLAMP3301H.TCT, U19 UCLAMP3301H.TCT, U2 UCLAMP3301H.TCT, U20 UCLAMP3301H.TCT, U21 RUC002N05T116, U3 UCLAMP3301H.TCT, U4 UCLAMP3301H.TCT, U5 UCLAMP3301H.TCT, U6 UCLAMP3301H.TCT, U7 JS102011SCQN, U8 UCLAMP3301H.TCT, U9 UCLAMP3301H.TCT

Commit message: Correct spacing on sensor board, refactor datasheets and project libraries
Parts:
- U1, U11, U12, U13, U14, U17, U18, U19, U2, U20, U3, U4, U5, U6, U8, U9: value UCLAMP3301H.TCT -> SOD_01H.TCT_SEM; footprint UCLAMP3310H-TCT:UCLAMP3301H.TCT -> UCLAMP3301H-TCT:UCLAMP3301H.TCT
- U21: value RUC002N05T116 -> SOT23-3_ROM; footprint RUC002N05116:RUC002N05T116 -> RUC002N05T116:RUC002N05T116

Commit message: adding 3w
Parts:
- renumbered TP14 to DNI, TP16 to DNI, TP17 to DNI, TP11 to DNI
