File: Boards/Sensor_Board_2x8/_Top_Level/Sensor_Board_2x8.kicad_pcb (KiCad board)
At the start: 2 copper layers, 95.3 x 406.4 mm, 34 parts, among them J1 OQ0212500000G, J10 OQ0212500000G, J11 OQ0212500000G, J12 OQ0212500000G, J13 OQ0212500000G, J14 OQ0212500000G, J15 OQ0212500000G, J16 OQ0212500000G, J17 OQ0212500000G, J18 OQ0212500000G, J2 OQ0212500000G, J3 OQ0212500000G, J4 OQ0212500000G, J5 OQ0212500000G, J6 OQ0212500000G, J7 OQ0212500000G, J8 OQ0212500000G, J9 OQ0212500000G

Commit message: Add mounting holes to sensor board
Parts:
- added ?: , , F.Cu at (111.0, 423.0)
- added REF**: MountingHole_5.3mm_M5_ISO7380_Pad, MountingHole:MountingHole_5.3mm_M5_ISO7380_Pad, F.Cu at (111.0, 33.6)
- added REF**: MountingHole_5.3mm_M5_ISO7380_Pad, MountingHole:MountingHole_5.3mm_M5_ISO7380_Pad, F.Cu at (32.8, 33.6)
- added REF**: MountingHole_5.3mm_M5_ISO7380_Pad, MountingHole:MountingHole_5.3mm_M5_ISO7380_Pad, F.Cu at (32.8, 423.0)
- moved J10 15.8 mm to (87.8, 426.9)
Routing:
- net Net-(J10-Pad1): track 758.8 -> 772.0 mm
Changed lines of the file:
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@@
     )
+  )
+  (footprint "MountingHole:MountingHole_5.3mm_M5_ISO7380_Pad" (layer "F.Cu")
+    (at 111.0424 33.6206)
+    (descr "Mounting Hole 5.3mm, M5, ISO7380")
+    (tags "mounting hole 5.3mm m5 iso7380")
+    (attr exclude_from_pos_files exclude_from_bom)
+    (fp_text reference "REF**" (at 0 -5.75) (layer "F.SilkS")
+      (effects (font (size 1 1) (thickness 0.15)))
+    )
+    (fp_text value "MountingHole_5.3mm_M5_ISO7380_Pad" (at 0 5.75) (layer "F.Fab") hide
+      (effects (font (size 1 1) (thickness 0.15)))
+    )
+    (fp_text user "${REFERENCE}" (at 0 0) (layer "F.Fab")
+      (effects (font (size 1 1) (thickness 0.15)))
+    )
+    (fp_circle (center 0 0) (end 4.75 0) (layer "Cmts.User") (width 0.15) (fill none))
+    (fp_circle (center 0 0) (end 5 0) (layer "F.CrtYd") (width 0.05) (fill none))
+    (pad "1" thru_hole circle (at 0 0) (size 9.5 9.5) (drill 5.3) (layers F&B.Cu *.Mask))
   )
   (footprint "GP560_V03:GP560_V03" (layer "F.Cu")
@@
     )
   )
+  (footprint "" (layer "F.Cu")
+    (at 111.0424 423.0206)
+    (fp_text reference "" (at 0 0) (layer "F.SilkS")
+      (effects (font (size 1.27 1.27) (thickness 0.15)))
+    )
+    (fp_text value "" (at 0 0) (layer "F.SilkS")
+      (effects (font (size 1.27 1.27) (thickness 0.15)))
+    )
+    (pad "1" thru_hole circle (at 0 0) (size 9.5 9.5) (drill 5.3) (layers F&B.Cu *.Mask))
+  )
   (footprint "OQ0212500000G:OQ0212500000G" (layer "F.Cu")
     (at 113.3244 390.7282 -90)
@@
       (rotate (xyz 0 0 0))
     )
+  )
+  (footprint "MountingHole:MountingHole_5.3mm_M5_ISO7380_Pad" (layer "F.Cu")
+    (at 32.7824 33.6206)
+    (descr "Mounting Hole 5.3mm, M5, ISO7380")
+    (tags "mounting hole 5.3mm m5 iso7380")
+    (attr exclude_from_pos_files exclude_from_bom)
+    (fp_text reference "REF**" (at 0 -5.75) (layer "F.SilkS")
+      (effects (font (size 1 1) (thickness 0.15)))
+    )
+    (fp_text value "MountingHole_5.3mm_M5_ISO7380_Pad" (at 0 5.75) (layer "F.Fab") hide
+      (effects (font (size 1 1) (thickness 0.15)))
+    )
+    (fp_text user "${REFERENCE}" (at 0 0) (layer "F.Fab")
+      (effects (font (size 1 1) (thickness 0.15)))
+    )
+    (fp_circle (center 0 0) (end 4.75 0) (layer "Cmts.User") (width 0.15) (fill none))
+    (fp_circle (center 0 0) (end 5 0) (layer "F.CrtYd") (width 0.05) (fill none))
+    (pad "1" thru_hole circle (at 0 0) (size 9.5 9.5) (drill 5.3) (layers F&B.Cu *.Mask))
   )
   (footprint "OQ0212500000G:OQ0212500000G" (layer "F.Cu")
@@
     )
   )
+  (footprint "MountingHole:MountingHole_5.3mm_M5_ISO7380_Pad" (layer "F.Cu")
+    (at 32.7824 423.0206)
+    (descr "Mounting Hole 5.3mm, M5, ISO7380")
+    (tags "mounting hole 5.3mm m5 iso7380")
+    (attr exclude_from_pos_files exclude_from_bom)
+    (fp_text reference "REF**" (at 0 -5.75) (layer "F.SilkS")
+      (effects (font (size 1 1) (thickness 0.15)))
+    )
+    (fp_text value "MountingHole_5.3mm_M5_ISO7380_Pad" (at 0 5.75) (layer "F.Fab") hide
+      (effects (font (size 1 1) (thickness 0.15)))
+    )
+    (fp_text user "${REFERENCE}" (at 0 0) (layer "F.Fab")
+      (effects (font (size 1 1) (thickness 0.15)))
+    )
+    (fp_circle (center 0 0) (end 4.75 0) (layer "Cmts.User") (width 0.15) (fill none))
+    (fp_circle (center 0 0) (end 5 0) (layer "F.CrtYd") (width 0.05) (fill none))
+    (pad "1" thru_hole circle (at 0 0) (size 9.5 9.5) (drill 5.3) (layers *.Cu *.Mask))
+  )
   (footprint "OQ0212500000G:OQ0212500000G" (layer "F.Cu")
     (at 28.5242 390.7282 -90)
@@
   )
   (footprint "OQ0212500000G:OQ0212500000G" (layer "F.Cu")
-    (at 103.6192 426.8596)
+    (at 87.8356 426.8596)
     (descr "OQ0212500000G-1")
     (tags "Connector")
@@
   (segment (start 65.6944 346.878968) (end 46.516232 346.878968) (width 0.762) (layer "B.Cu") (net 9))
   (segment (start 46.516232 346.912368) (end 46.516232 346.878968) (width 0.762) (layer "B.Cu") (net 9))
-  (segment (start 107.1192 48.1778) (end 107.11 48.1686) (width 0.762) (layer "F.Cu") (net 10))
-  (segment (start 107.1192 426.8596) (end 107.1192 48.1778) (width 0.762) (layer "F.Cu") (net 10))
+  (segment (start 107.11 411.0852) (end 107.11 48.1686) (width 0.762) (layer "F.Cu") (net 10))
+  (segment (start 87.8356 426.8596) (end 87.9222 426.8596) (width 0.762) (layer "F.Cu") (net 10))
+  (segment (start 91.3356 426.8596) (end 107.11 411.0852) (width 0.762) (layer "F.Cu") (net 10))
+  (segment (start 103.6192 411.1626) (end 103.6192 51.6594) (width 0.762) (layer "F.Cu") (net 10))
   (segment (start 103.6192 51.6594) (end 107.11 48.1686) (width 0.762) (layer "F.Cu") (net 10))
-  (segment (start 103.6192 426.8596) (end 103.6192 51.6594) (width 0.762) (layer "F.Cu") (net 10))
+  (segment (start 87.9222 426.8596) (end 103.6192 411.1626) (width 0.762) (layer "F.Cu") (net 10))
   (segment (start 76.1542 390.7282) (end 113.3244 390.7282) (width 0.762) (layer "B.Cu") (net 11))
   (segment (start 65.6944 390.7282) (end 76.1542 390.7282) (width 0.762) (layer "B.Cu") (net 11))

Commit message: Adjust sensor board width
Parts:
- moved ? 2.54 mm to (108.5, 423.0)
- moved REF** 2.54 mm to (108.5, 33.6)
- moved J11 2.54 mm to (110.8, 59.3)
- moved J12 2.54 mm to (110.8, 106.6)
- moved J13 2.54 mm to (110.8, 154.0)
- moved J14 2.54 mm to (110.8, 201.3)
- moved J15 2.54 mm to (110.8, 248.7)
- moved J16 2.54 mm to (110.8, 296.0)
- moved J17 2.54 mm to (110.8, 343.4)
- moved J18 2.54 mm to (110.8, 390.7)
- moved S1 1.27 mm to (31.3, 75.0)
- moved S2 1.27 mm to (31.3, 122.7)
- moved S3 1.27 mm to (31.3, 170.3)
- moved S4 1.27 mm to (31.3, 217.9)
- moved S5 1.27 mm to (31.3, 265.6)
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Routing:
- net Net-(J18-Pad2): track 124.9 -> 122.4 mm
- net Net-(J1-Pad2): track 119.6 -> 117.1 mm
- net Net-(J18-Pad1): track 84.8 -> 82.3 mm
- net Net-(J17-Pad2): track 124.2 -> 121.7 mm
- net Net-(J17-Pad1): track 84.8 -> 82.3 mm
- net Net-(J16-Pad2): track 123.7 -> 121.2 mm
- net Net-(J16-Pad1): track 84.8 -> 82.3 mm
- net Net-(J15-Pad2): track 122.6 -> 120.1 mm
- net Net-(J15-Pad1): track 84.8 -> 82.3 mm
- net Net-(J14-Pad2): track 121.8 -> 119.2 mm
- net Net-(J14-Pad1): track 84.8 -> 82.3 mm
- net Net-(J13-Pad2): track 121.2 -> 118.6 mm
- net Net-(J13-Pad1): track 84.8 -> 82.3 mm
- net Net-(J12-Pad2): track 120.4 -> 117.9 mm
- net Net-(J12-Pad1): track 84.8 -> 82.3 mm
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Other:
- board size 95.3 x 406.4 mm -> 92.7 x 406.4 mm

Commit message: Enlargen sensor board pads
Parts:
- J1, J10, J11, J12, J13, J14, J15, J16, J17, J18, J2, J3, J4, J5, J6, J7, J8, J9: value OQ0212500000G -> OQ0212500000G_Big_Pad; footprint OQ0212500000G:OQ0212500000G -> OQ0212500000G:OQ0212500000G_Big_Pad

Commit message: sizing of assembly pdf
Parts:
- J1, J10, J11, J12, J13, J14, J15, J16, J17, J18, J2, J3, J4, J5, J6, J7, J8, J9: value OQ0212500000G_Big_Pad -> OQ0212500000G; footprint OQ0212500000G:OQ0212500000G_Big_Pad -> OQ0212500000G:OQ0212500000G
