File: Boards/Main_Board/Sensor_Subsystem/SensorNetwork.kicad_sch (KiCad schematic)
At the start: 34 parts, among them J12 OQ0432500000G, J13 OQ0432500000G, J14 OQ0432500000G, J15 OQ0432500000G, J16 OQ0432500000G, J17 OQ0432500000G, J18 OQ0432500000G, J19 OQ0432500000G, U13 UCLAMP3301H.TCT, U14 UCLAMP3301H.TCT, U15 SN74LV4051ATPWRQ1, U16 SN74LV4051ATPWRQ1

Commit message: Correct spacing on sensor board, refactor datasheets and project libraries
Parts:
- C33, C34: symbol CL10B104KB8NNC:CL10B104KB8NNNC -> CL10B104KB8NNNC:CL10B104KB8NNNC
- J12, J13, J14, J15, J16, J17, J18, J19: symbol OQ04325500000G:OQ0432500000G -> OQ0432500000G:OQ0432500000G
Changed lines of the file:
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@@
     (pin "1")
   )
-  (symbol (lib_id "CL10B104KB8NNC:CL10B104KB8NNNC") (at 77.47 118.11 90) (mirror x) (unit 1)
+  (symbol (lib_id "CL10B104KB8NNNC:CL10B104KB8NNNC") (at 77.47 118.11 90) (mirror x) (unit 1)
     (in_bom yes) (on_board yes)
     (property "Reference" "C34" (id 0) (at 83.82 119.38 90)
@@
     (pin "2")
   )
-  (symbol (lib_id "OQ04325500000G:OQ0432500000G") (at 151.13 60.96 0) (unit 1)
+  (symbol (lib_id "OQ0432500000G:OQ0432500000G") (at 151.13 60.96 0) (unit 1)
     (in_bom yes) (on_board yes) (fields_autoplaced)
     (property "Reference" "J12" (id 0) (at 167.64 64.7699 0)
@@
       (effects (font (size 1.27 1.27)) hide)
     )
-    (property "Manufacturer's Part Number" "OQ0432500000G" (id 14) (at 151.13 60.96 0)
-      (effects (font (size 1.27 1.27)) hide)
+    (property "Manufacturer's Part Number" "OQ0432500000G" (id 14) (at 167.64 76.2 0)
+      (effects (font (size 1.27 1.27)) (justify left) hide)
     )
     (pin "1")
@@
     (pin "2")
   )
-  (symbol (lib_id "UCLAMP3301H-TCT:UCLAMP3301H.TCT") (at 49.53 166.37 90) (unit 1)
+  (symbol (lib_name "UCLAMP3301H.TCT_1") (lib_id "UCLAMP3301H-TCT:UCLAMP3301H.TCT") (at 49.53 166.37 90) (unit 1)
     (in_bom yes) (on_board yes)
     (property "Reference" "U14" (id 0) (at 55.88 149.86 90)
@@
     (pin "9")
   )
-  (symbol (lib_id "OQ04325500000G:OQ0432500000G") (at 151.13 127 0) (unit 1)
+  (symbol (lib_id "OQ0432500000G:OQ0432500000G") (at 151.13 127 0) (unit 1)
     (in_bom yes) (on_board yes) (fields_autoplaced)
     (property "Reference" "J14" (id 0) (at 167.64 130.8099 0)
@@
       (effects (font (size 1.27 1.27)) hide)
     )
-    (property "Manufacturer's Part Number" "OQ0432500000G" (id 14) (at 151.13 127 0)
-      (effects (font (size 1.27 1.27)) hide)
+    (property "Manufacturer's Part Number" "OQ0432500000G" (id 14) (at 167.64 142.24 0)
+      (effects (font (size 1.27 1.27)) (justify left) hide)
     )
     (pin "1")
@@
     (pin "2")
   )
-  (symbol (lib_id "OQ04325500000G:OQ0432500000G") (at 151.13 139.7 0) (unit 1)
+  (symbol (lib_id "OQ0432500000G:OQ0432500000G") (at 151.13 139.7 0) (unit 1)
     (in_bom yes) (on_board yes) (fields_autoplaced)
     (property "Reference" "J15" (id 0) (at 167.64 142.2399 0)
@@
       (effects (font (size 1.27 1.27)) hide)
     )
-    (property "Manufacturer's Part Number" "OQ0432500000G" (id 14) (at 151.13 139.7 0)
-      (effects (font (size 1.27 1.27)) hide)
+    (property "Manufacturer's Part Number" "OQ0432500000G" (id 14) (at 167.64 154.94 0)
+      (effects (font (size 1.27 1.27)) (justify left) hide)
     )
     (pin "1")
@@
     (pin "1")
   )
-  (symbol (lib_id "OQ04325500000G:OQ0432500000G") (at 248.92 135.89 90) (unit 1)
+  (symbol (lib_id "OQ0432500000G:OQ0432500000G") (at 248.92 135.89 90) (unit 1)
     (in_bom yes) (on_board yes) (fields_autoplaced)
     (property "Reference" "J19" (id 0) (at 251.4599 119.38 0)
@@
       (effects (font (size 1.27 1.27)) hide)
     )
-    (property "Manufacturer's Part Number" "OQ0432500000G" (id 14) (at 248.92 135.89 0)
-      (effects (font (size 1.27 1.27)) hide)
+    (property "Manufacturer's Part Number" "OQ0432500000G" (id 14) (at 264.16 119.38 0)
+      (effects (font (size 1.27 1.27)) (justify left) hide)
     )
     (pin "1")
@@
     (pin "2")
   )
-  (symbol (lib_id "OQ04325500000G:OQ0432500000G") (at 204.47 135.89 90) (unit 1)
+  (symbol (lib_id "OQ0432500000G:OQ0432500000G") (at 204.47 135.89 90) (unit 1)
     (in_bom yes) (on_board yes) (fields_autoplaced)
     (property "Reference" "J17" (id 0) (at 207.0099 119.38 0)
@@
       (effects (font (size 1.27 1.27)) hide)
     )
-    (property "Manufacturer's Part Number" "OQ0432500000G" (id 14) (at 204.47 135.89 0)
-      (effects (font (size 1.27 1.27)) hide)
+    (property "Manufacturer's Part Number" "OQ0432500000G" (id 14) (at 219.71 119.38 0)
+      (effects (font (size 1.27 1.27)) (justify left) hide)
     )
     (pin "1")
@@
     (pin "4")
   )
-  (symbol (lib_id "OQ04325500000G:OQ0432500000G") (at 248.92 71.12 90) (unit 1)
+  (symbol (lib_id "OQ0432500000G:OQ0432500000G") (at 248.92 71.12 90) (unit 1)
     (in_bom yes) (on_board yes) (fields_autoplaced)
     (property "Reference" "J18" (id 0) (at 251.4599 54.61 0)
@@
       (effects (font (size 1.27 1.27)) hide)
     )
-    (property "Manufacturer's Part Number" "OQ0432500000G" (id 14) (at 248.92 71.12 0)
-      (effects (font (size 1.27 1.27)) hide)
+    (property "Manufacturer's Part Number" "OQ0432500000G" (id 14) (at 264.16 54.61 0)
+      (effects (font (size 1.27 1.27)) (justify left) hide)
     )
     (pin "1")
@@
     (pin "2")
   )
-  (symbol (lib_id "OQ04325500000G:OQ0432500000G") (at 151.13 73.66 0) (unit 1)
+  (symbol (lib_id "OQ0432500000G:OQ0432500000G") (at 151.13 73.66 0) (unit 1)
     (in_bom yes) (on_board yes) (fields_autoplaced)
     (property "Reference" "J13" (id 0) (at 167.64 76.1999 0)
@@
       (effects (font (size 1.27 1.27)) hide)
     )
-    (property "Manufacturer's Part Number" "OQ0432500000G" (id 14) (at 151.13 73.66 0)
-      (effects (font (size 1.27 1.27)) hide)
+    (property "Manufacturer's Part Number" "OQ0432500000G" (id 14) (at 167.64 88.9 0)
+      (effects (font (size 1.27 1.27)) (justify left) hide)
     )
     (pin "1")
@@
     (pin "2")
   )
-  (symbol (lib_id "CL10B104KB8NNC:CL10B104KB8NNNC") (at 77.47 52.07 90) (mirror x) (unit 1)
+  (symbol (lib_id "CL10B104KB8NNNC:CL10B104KB8NNNC") (at 77.47 52.07 90) (mirror x) (unit 1)
     (in_bom yes) (on_board yes)
     (property "Reference" "C33" (id 0) (at 83.82 53.34 90)
@@
     (pin "2")
   )
-  (symbol (lib_id "OQ04325500000G:OQ0432500000G") (at 204.47 71.12 90) (unit 1)
+  (symbol (lib_id "OQ0432500000G:OQ0432500000G") (at 204.47 71.12 90) (unit 1)
     (in_bom yes) (on_board yes) (fields_autoplaced)
     (property "Reference" "J16" (id 0) (at 207.0099 54.61 0)
@@
       (effects (font (size 1.27 1.27)) hide)
     )
-    (property "Manufacturer's Part Number" "OQ0432500000G" (id 14) (at 204.47 71.12 0)
-      (effects (font (size 1.27 1.27)) hide)
-    )
-    (pin "1")
+    (property "Manufacturer's Part Number" "OQ0432500000G" (id 14) (at 219.71 54.61 0)
+      (effects (font (size 1.27 1.27)) (justify left) hide)
+    )
+    (pin "1")

Commit message: Changes for sensor network
Other:
- note added: "DEMUX (Select Row)"
- note added: "MUX (Select Column)"
- note removed: "DEMUX (Select Column)"
Changed lines of the file:
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@@
     (stroke (width 0) (type default) (color 0 0 0 0))
   )
-  (text "DEMUX (Select Column)" (at 30.48 45.72 0)
+  (text "MUX (Select Column)" (at 30.48 45.72 0)
     (effects (font (size 1.27 1.27) (thickness 0.254) bold) (justify left bottom))
   )
-  (text "General Notes:\n	Assumes a crosspoint array of 8 rows, 8 columns, connected by reed switches\n	Reed switches to be used - https://standexelectronics.com/viewer/pdfjs/web/viewer.php?file=https%3A%2F%2Fstandexelectronics.com%2Fwp-content%2Fuploads%2F2019%2F06%2FGP560_V03.pdf\n	DEMUX selects the column to be sent power\n	MUX selects the row to read\n	Designed for carry current of 6mA\n	*** BE MINDFUL OF THE ORDERING OF CONNECTOR PINS ***"
-    (at 16.51 29.21 0)
+  (text "General Notes:\n	Assumes a crosspoint array of 8 rows, 8 columns, connected by reed switches\n	Reed switches to be used - https://standexelectronics.com/viewer/pdfjs/web/viewer.php?file=https%3A%2F%2Fstandexelectronics.com%2Fwp-content%2Fuploads%2F2019%2F06%2FGP560_V03.pdf\n	DEMUX selects the column to be sent power\n	MUX selects the row to read\n	Designed for carry current of 6mA\n	*** BE MINDFUL OF THE ORDERING OF CONNECTOR PINS ***\n\nWARNING: There is a mistake on the DEMUX, VCC and COM should be separate"
+    (at 16.51 33.02 0)
     (effects (font (size 1.27 1.27)) (justify left bottom))
   )
-  (text "DEMUX (Select Column)" (at 30.48 111.76 0)
+  (text "DEMUX (Select Row)" (at 30.48 111.76 0)
     (effects (font (size 1.27 1.27) (thickness 0.254) bold) (justify left bottom))
   )

Commit message: Fix typos
Other:
- note added: "DEMUX (Select Column)"
- note added: "MUX (Select Row)"
- note removed: "DEMUX (Select Row)"
- note removed: "MUX (Select Column)"
Changed lines of the file:
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@@
     (stroke (width 0) (type default) (color 0 0 0 0))
   )
-  (text "MUX (Select Column)" (at 30.48 45.72 0)
+  (text "DEMUX (Select Column)" (at 30.48 45.72 0)
     (effects (font (size 1.27 1.27) (thickness 0.254) bold) (justify left bottom))
   )
@@
     (effects (font (size 1.27 1.27)) (justify left bottom))
   )
-  (text "DEMUX (Select Row)" (at 30.48 111.76 0)
+  (text "MUX (Select Row)" (at 30.48 111.76 0)
     (effects (font (size 1.27 1.27) (thickness 0.254) bold) (justify left bottom))
   )
