File: Boards/Sensor_Board_4x16/_Top_Level/Sensor_Board_4x16.kicad_pcb (KiCad board)
At the start: 2 copper layers, 92.7 x 406.4 mm, 38 parts, among them J1 OQ0212500000G, J10 OQ0212500000G, J11 OQ0212500000G, J12 OQ0212500000G, J13 OQ0212500000G, J14 OQ0212500000G, J15 OQ0212500000G, J16 OQ0212500000G, J17 OQ0212500000G, J18 OQ0212500000G, J2 OQ0212500000G, J3 OQ0212500000G, J4 OQ0212500000G, J5 OQ0212500000G, J6 OQ0212500000G, J7 OQ0212500000G, J8 OQ0212500000G, J9 OQ0212500000G

Commit message: Fix typos
Parts:
- added REF**: D_MELF, Diode_SMD:D_MELF, F.Cu at (31.4, 402.5)
- added REF**: D_MELF, Diode_SMD:D_MELF, F.Cu at (91.5, 408.3)
Routing:
- net Net-(J18-Pad2): track 122.4 -> 126.1 mm
Changed lines of the file:
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@@
+    )
+  )
+  (footprint "Diode_SMD:D_MELF" (layer "F.Cu")
+    (at 31.4198 402.5392 -90)
+    (descr "Diode, MELF,,")
+    (tags "Diode MELF ")
+    (attr smd)
+    (fp_text reference "REF**" (at 0 -2.5 90) (layer "F.SilkS")
+      (effects (font (size 1 1) (thickness 0.15)))
+    )
+    (fp_text value "D_MELF" (at -0.25 2.5 90) (layer "F.Fab")
+      (effects (font (size 1 1) (thickness 0.15)))
+    )
+    (fp_text user "${REFERENCE}" (at 0 -2.5 90) (layer "F.Fab")
+      (effects (font (size 1 1) (thickness 0.15)))
+    )
+    (fp_line (start -3.3 -1.5) (end -3.3 1.5) (layer "F.SilkS") (width 0.12))
+    (fp_line (start 2.4 -1.5) (end -3.3 -1.5) (layer "F.SilkS") (width 0.12))
+    (fp_line (start -3.3 1.5) (end 2.4 1.5) (layer "F.SilkS") (width 0.12))
+    (fp_line (start 3.4 -1.6) (end 3.4 1.6) (layer "F.CrtYd") (width 0.05))
+    (fp_line (start -3.4 1.6) (end -3.4 -1.6) (layer "F.CrtYd") (width 0.05))
+    (fp_line (start 3.4 1.6) (end -3.4 1.6) (layer "F.CrtYd") (width 0.05))
+    (fp_line (start -3.4 -1.6) (end 3.4 -1.6) (layer "F.CrtYd") (width 0.05))
+    (fp_line (start -0.64944 0.00102) (end 0.50118 -0.79908) (layer "F.Fab") (width 0.1))
+    (fp_line (start 2.6 -1.3) (end -2.6 -1.3) (layer "F.Fab") (width 0.1))
+    (fp_line (start -0.64944 -0.79908) (end -0.64944 0.80112) (layer "F.Fab") (width 0.1))
+    (fp_line (start -2.6 1.3) (end 2.6 1.3) (layer "F.Fab") (width 0.1))
+    (fp_line (start -0.64944 0.00102) (end 0.50118 0.75032) (layer "F.Fab") (width 0.1))
+    (fp_line (start -0.64944 0.00102) (end -1.55114 0.00102) (layer "F.Fab") (width 0.1))
+    (fp_line (start -2.6 -1.3) (end -2.6 1.3) (layer "F.Fab") (width 0.1))
+    (fp_line (start 0.50118 0.75032) (end 0.50118 -0.79908) (layer "F.Fab") (width 0.1))
+    (fp_line (start 2.6 1.3) (end 2.6 -1.3) (layer "F.Fab") (width 0.1))
+    (fp_line (start 0.50118 0.00102) (end 1.4994 0.00102) (layer "F.Fab") (width 0.1))
+    (pad "1" smd rect (at -2.4 0 270) (size 1.5 2.7) (layers "F.Cu" "F.Paste" "F.Mask")
+      (net 17 "Net-(J18-Pad2)"))
+    (pad "2" smd rect (at 2.4 0 270) (size 1.5 2.7) (layers "F.Cu" "F.Paste" "F.Mask")
+      (net 17 "Net-(J18-Pad2)"))
+    (model "${KICAD6_3DMODEL_DIR}/Diode_SMD.3dshapes/D_MELF.wrl"
+      (offset (xyz 0 0 0))
+      (scale (xyz 1 1 1))
+      (rotate (xyz 0 0 0))
     )
   )
@@
     (pad "1" thru_hole circle (at 0 0) (size 9.5 9.5) (drill 5.3) (layers F&B.Cu *.Mask))
   )
+  (footprint "Diode_SMD:D_MELF" (layer "F.Cu")
+    (at 91.4654 408.3304 180)
+    (descr "Diode, MELF,,")
+    (tags "Diode MELF ")
+    (attr smd)
+    (fp_text reference "REF**" (at 0 -2.5) (layer "F.SilkS")
+      (effects (font (size 1 1) (thickness 0.15)))
+    )
+    (fp_text value "D_MELF" (at -0.25 2.5) (layer "F.Fab")
+      (effects (font (size 1 1) (thickness 0.15)))
+    )
+    (fp_text user "${REFERENCE}" (at 0 -2.5) (layer "F.Fab")
+      (effects (font (size 1 1) (thickness 0.15)))
+    )
+    (fp_line (start -3.3 -1.5) (end -3.3 1.5) (layer "F.SilkS") (width 0.12))
+    (fp_line (start 2.4 -1.5) (end -3.3 -1.5) (layer "F.SilkS") (width 0.12))
+    (fp_line (start -3.3 1.5) (end 2.4 1.5) (layer "F.SilkS") (width 0.12))
+    (fp_line (start 3.4 -1.6) (end 3.4 1.6) (layer "F.CrtYd") (width 0.05))
+    (fp_line (start -3.4 1.6) (end -3.4 -1.6) (layer "F.CrtYd") (width 0.05))
+    (fp_line (start 3.4 1.6) (end -3.4 1.6) (layer "F.CrtYd") (width 0.05))
+    (fp_line (start -3.4 -1.6) (end 3.4 -1.6) (layer "F.CrtYd") (width 0.05))
+    (fp_line (start -0.64944 0.00102) (end 0.50118 -0.79908) (layer "F.Fab") (width 0.1))
+    (fp_line (start 2.6 -1.3) (end -2.6 -1.3) (layer "F.Fab") (width 0.1))
+    (fp_line (start -0.64944 -0.79908) (end -0.64944 0.80112) (layer "F.Fab") (width 0.1))
+    (fp_line (start -2.6 1.3) (end 2.6 1.3) (layer "F.Fab") (width 0.1))
+    (fp_line (start -0.64944 0.00102) (end 0.50118 0.75032) (layer "F.Fab") (width 0.1))
+    (fp_line (start -0.64944 0.00102) (end -1.55114 0.00102) (layer "F.Fab") (width 0.1))
+    (fp_line (start -2.6 -1.3) (end -2.6 1.3) (layer "F.Fab") (width 0.1))
+    (fp_line (start 0.50118 0.75032) (end 0.50118 -0.79908) (layer "F.Fab") (width 0.1))
+    (fp_line (start 2.6 1.3) (end 2.6 -1.3) (layer "F.Fab") (width 0.1))
+    (fp_line (start 0.50118 0.00102) (end 1.4994 0.00102) (layer "F.Fab") (width 0.1))
+    (pad "1" smd rect (at -2.4 0 180) (size 1.5 2.7) (layers "F.Cu" "F.Paste" "F.Mask")
+      (net 17 "Net-(J18-Pad2)"))
+    (pad "2" smd rect (at 2.4 0 180) (size 1.5 2.7) (layers "F.Cu" "F.Paste" "F.Mask")
+      (net 17 "Net-(J18-Pad2)"))
+    (model "${KICAD6_3DMODEL_DIR}/Diode_SMD.3dshapes/D_MELF.wrl"
+      (offset (xyz 0 0 0))
+      (scale (xyz 1 1 1))
+      (rotate (xyz 0 0 0))
+    )
+  )
   (footprint "GP560_V03:GP560_V03" (layer "F.Cu")
     (at 31.34 408.4486)
@@
     (pts (xy 24.2824 431.5206) (xy 117.0024 431.5206))
     (height 2.9972)
-    (gr_text "3.6504 in" (at 70.6424 433.3678) (layer "F.Fab")
+    (gr_text "92.7200 mm" (at 70.6424 433.3678) (layer "F.Fab")
       (effects (font (size 1 1) (thickness 0.15)))
     )
@@
     (pts (xy 117.0024 431.5206) (xy 117.0024 25.1206))
     (height 3.3782)
-    (gr_text "16.0000 in" (at 119.2306 228.3206 90) (layer "F.Fab")
+    (gr_text "406.4000 mm" (at 119.2306 228.3206 90) (layer "F.Fab")
       (effects (font (size 1 1) (thickness 0.15)))
     )
@@
   (segment (start 28.5242 248.680512) (end 110.7844 248.680512) (width 0.762) (layer "B.Cu") (net 15))
   (segment (start 28.5242 296.02974) (end 110.7844 296.02974) (width 0.762) (layer "B.Cu") (net 16))
+  (segment (start 89.0654 408.3304) (end 79.0882 408.3304) (width 0.25) (layer "F.Cu") (net 17))
+  (segment (start 31.4198 408.3688) (end 31.34 408.4486) (width 0.25) (layer "F.Cu") (net 17))
+  (segment (start 79.0882 408.3304) (end 78.97 408.4486) (width 0.25) (layer "F.Cu") (net 17))
+  (segment (start 31.4198 404.9392) (end 31.4198 408.3688) (width 0.25) (layer "F.Cu") (net 17))
+  (segment (start 96.8854 408.1272) (end 94.0054 408.1272) (width 0.762) (layer "B.Cu") (net 17))
   (segment (start 74.8842 394.2282) (end 64.4244 394.2282) (width 0.762) (layer "B.Cu") (net 17))
+  (segment (start 31.3944 397.0984) (end 31.3944 400.304) (width 0.762) (layer "B.Cu") (net 17))
   (segment (start 110.7844 394.2282) (end 93.0908 394.2282) (width 0.762) (layer "B.Cu") (net 17))
-  (segment (start 31.34 408.4486) (end 45.4608 394.3278) (width 0.762) (layer "B.Cu") (net 17))
   (segment (start 45.4608 394.3278) (end 45.4608 394.2282) (width 0.762) (layer "B.Cu") (net 17))
+  (segment (start 110.7844 394.2282) (end 96.8854 408.1272) (width 0.762) (layer "B.Cu") (net 17))
+  (segment (start 28.5242 394.2282) (end 31.3944 397.0984) (width 0.762) (layer "B.Cu") (net 17))
+  (segment (start 94.0054 408.1272) (end 93.9038 408.2288) (width 0.762) (layer "B.Cu") (net 17))
   (segment (start 45.4608 394.2282) (end 28.5242 394.2282) (width 0.762) (layer "B.Cu") (net 17))
   (segment (start 93.0908 394.2282) (end 74.8842 394.2282) (width 0.762) (layer "B.Cu") (net 17))
   (segment (start 64.4244 394.2282) (end 45.4608 394.2282) (width 0.762) (layer "B.Cu") (net 17))
-  (segment (start 78.97 408.4486) (end 93.0908 394.3278) (width 0.762) (layer "B.Cu") (net 17))
   (segment (start 93.0908 394.3278) (end 93.0908 394.2282) (width 0.762) (layer "B.Cu") (net 17))
   (segment (start 58.2192 48.1778) (end 58.21 48.1686) (width 0.762) (layer "F.Cu") (net 18))
